Commit message: lost track

File: ros_ws/src/simplebot_description/urdf/roarm_m2/roarm_m2.xacro (robot description, xacro)
@@ -141,5 +141,5 @@
 <!-- Fixed joint placing tool0 at the end of link3 (the tool mounting point) -->
 <joint name="link4_to_link5" type="revolute">
-  <origin xyz="0.09187 0.0079 -0.00078" rpy="0 1.5708 0" />
+  <origin xyz="0.09387 0.0079 -0.00078" rpy="0 1.5708 0" />
   <parent link="link4" />
   <child link="link5" />
@@ -148,5 +148,5 @@
 </joint>
 <joint name="link4_to_tool0" type="fixed">
-  <origin xyz="0.09187 0.0079 -0.00078" rpy="0 1.5708 0" />
+  <origin xyz="0.09387 0.0079 -0.00078" rpy="0 1.5708 0" />
   <parent link="link4" />
   <child link="tool0" />
