Commit message: changes

File: ros_ws/src/simplebot_description/urdf/control_m2/roarm_m2.ros2_control.xacro (robot description, xacro)
@@ -35,10 +35,47 @@
                 <state_interface name="velocity"/>
             </joint>
-            <joint name="link3_to_gripper_link">
+            <joint name="link3_to_link4">
                 <command_interface name="position"/>
                 <state_interface name="position">
-                  <param name="initial_value">${initial_positions['link3_to_gripper_link']}</param>
+                  <param name="initial_value">${initial_positions['link3_to_link4']}</param>
                 </state_interface>
                 <state_interface name="velocity"/>
+            </joint>
+            <joint name="link4_to_link5">
+                <command_interface name="position"/>
+                <state_interface name="position">
+                  <param name="initial_value">${initial_positions['link4_to_link5']}</param>
+                </state_interface>
+                <state_interface name="velocity"/>
+            </joint>
+            <joint name="straight_bracket_left_joint">
+            <command_interface name="position"/>
+            <state_interface name="position"/>
+            <state_interface name="velocity"/>
+            </joint>
+            <joint name="straight_bracket_right_joint">
+            <param name="mimic">straight_bracket_left_joint</param>
+            <param name="multiplier">-1.0</param>
+            <state_interface name="position"/>
+            </joint>
+            <joint name="left_gear_arm_joint">
+            <param name="mimic">straight_bracket_left_joint</param>
+            <param name="multiplier">1.0</param>
+            <state_interface name="position"/>
+            </joint>
+            <joint name="right_gear_arm_joint">
+            <param name="mimic">straight_bracket_left_joint</param>
+            <param name="multiplier">-1.0</param>
+            <state_interface name="position"/>
+            </joint>
+            <joint name="left_finger_joint">
+            <param name="mimic">straight_bracket_left_joint</param>
+            <param name="multiplier">-1.0</param>
+            <state_interface name="position"/>
+            </joint>
+            <joint name="right_finger_joint">
+            <param name="mimic">straight_bracket_left_joint</param>
+            <param name="multiplier">1.0</param>
+            <state_interface name="position"/>
             </joint>
         </ros2_control>

File: ros_ws/src/simplebot_description/urdf/femto_bolt/femto_bolt.urdf.xacro (robot description, xacro)
@@ -29,5 +29,5 @@
         <origin xyz="0 0 0" rpy="0 0 0"/>
         <geometry>
-          <mesh filename="$(find simplebot_description)/meshes/femto_bolt/femto_bolt.stl" />
+          <mesh filename="package://simplebot_description/meshes/femto_bolt/femto_bolt.stl" />
         </geometry>
         <material name="">
@@ -37,7 +37,7 @@
       <collision>
         <origin xyz="0 0 0" rpy="0 0 0"/>
-        <geometry>
-          <mesh filename="$(find simplebot_description)/meshes/femto_bolt/femto_bolt.stl" />
-        </geometry>
+          <geometry>
+            <mesh filename="package://simplebot_description/meshes/femto_bolt/femto_bolt.stl" />
+          </geometry>
       </collision>
       <inertial>

File: ros_ws/src/simplebot_description/urdf/roarm_m2/roarm_m2.xacro (robot description, xacro)
@@ -4,4 +4,6 @@
 <xacro:include filename="$(find simplebot_description)/urdf/roarm_m2/roarm_m2.trans" />
 <xacro:include filename="$(find simplebot_description)/urdf/roarm_m2/roarm_m2.gazebo" />
+<xacro:include filename="$(find simplebot_description)/urdf/roarm_m2/gripper.xacro" />
+<!-- ===== ARM LINKS ===== -->
 <link name="roarm_base_link">
   <inertial>
@@ -84,88 +86,11 @@
   </collision>
 </link>
-<link name="gripper_link">
+<!-- tool0: the tool mounting frame at the end of link3.
+     This is where the gripper attaches. -->
+<link name="tool0" />
+<link name="link5" />
+<link name="link4">
   <inertial>
     <origin xyz="0.029 0.0027 -0.00078" rpy="0 0 0" />
-    <mass value="0.0028708" />
-    <inertia ixx="5.23216E-07" ixy="0" ixz="0" iyy="1.82071E-06" iyz="0" izz="1.60231E-06" />
-  </inertial>
-  <visual>
-    <origin xyz="0 0 0" rpy="0 0 0" />
-    <geometry>
-      <mesh filename="file://$(find simplebot_description)/meshes/roarm_m2/gripper_link.stl"  scale="1.0 1.0 1.0"/>
-    </geometry>
-    <material name="silver"/>
-  </visual>
-  <collision>
-    <origin xyz="0 0 0" rpy="0 0 0" />
-    <geometry>
-      <mesh filename="file://$(find simplebot_description)/meshes/roarm_m2/gripper_link.stl"  scale="1.0 1.0 1.0"/>
-    </geometry>
-  </collision>
-</link>
-<link name="gripper_b">
-  <inertial>
-    <origin xyz="0.029 0.0027 -0.00078" rpy="0 0 0" />
-    <mass value="0.0028708" />
-    <inertia ixx="5.23216E-07" ixy="0" ixz="0" iyy="1.82071E-06" iyz="0" izz="1.60231E-06" />
-  </inertial>
-  <visual>
-    <origin xyz="0 0 0" rpy="0 0 0" />
-    <geometry>
-      <mesh filename="file://$(find simplebot_description)/meshes/roarm_m2/Gripper-B.stl"  scale="1.0 1.0 1.0"/>
-    </geometry>
-    <material name="silver"/>
-  </visual>
-  <collision>
-    <origin xyz="0 0 0" rpy="0 0 0" />
-    <geometry>
-      <mesh filename="file://$(find simplebot_description)/meshes/roarm_m2/Gripper-B.stl"  scale="1.0 1.0 1.0"/>
-    </geometry>
-  </collision>
-</link>
-<link name="left_finger">
-  <inertial>
-    <origin xyz="0.0 0.0 -0.0" rpy="0 0 0" />
-    <mass value="0.0028708" />
-    <inertia ixx="5.23216E-07" ixy="0" ixz="0" iyy="1.82071E-06" iyz="0" izz="1.60231E-06" />
-  </inertial>
-  <visual>
-    <origin xyz="0 0 0" rpy="0 0 0" />
-    <geometry>
-      <mesh filename="file://$(find simplebot_description)/meshes/roarm_m2/left_finger.stl"  scale="1.0 1.0 1.0"/>
-    </geometry>
-    <material name="silver"/>
-  </visual>
-  <collision>
-    <origin xyz="0 0 0" rpy="0 0 0" />
-    <geometry>
-      <mesh filename="file://$(find simplebot_description)/meshes/roarm_m2/left_finger.stl"  scale="1.0 1.0 1.0"/>
-    </geometry>
-  </collision>
-</link>
-<link name="right_finger">
-  <inertial>
-    <origin xyz="0.0 0.0 -0.0" rpy="0 0 0" />
-    <mass value="0.0028708" />
-    <inertia ixx="5.23216E-07" ixy="0" ixz="0" iyy="1.82071E-06" iyz="0" izz="1.60231E-06" />
-  </inertial>
-  <visual>
-    <origin xyz="0 0 0" rpy="0 0 0" />
-    <geometry>
-      <mesh filename="file://$(find simplebot_description)/meshes/roarm_m2/right_finger.stl"  scale="1.0 1.0 1.0"/>
-    </geometry>
-    <material name="silver"/>
-  </visual>
-  <collision>
-    <origin xyz="0 0 0" rpy="0 0 0" />
-    <geometry>
-      <mesh filename="file://$(find simplebot_description)/meshes/roarm_m2/right_finger.stl"  scale="1.0 1.0 1.0"/>
-    </geometry>
-  </collision>
-</link>
-<!--
-<link name="link4">
-  <inertial>
-    <origin xyz="0.024599 0 0.026788" rpy="0 0 0" />
     <mass value="0.0028708" />
     <inertia ixx="5.23216E-07" ixy="0" ixz="0" iyy="1.82071E-06" iyz="0" izz="1.60231E-06" />
@@ -185,45 +110,5 @@
   </collision>
 </link>
-<link name="link5">
-  <inertial>
-    <origin xyz="0.0 0 0.0" rpy="0 0 0" />
-    <mass value="0.0028708" />
-    <inertia ixx="5.23216E-07" ixy="0" ixz="0" iyy="1.82071E-06" iyz="0" izz="1.60231E-06" />
-  </inertial>
-  <visual>
-    <origin xyz="0 0 0" rpy="0 0 0" />
-    <geometry>
-      <mesh filename="file://$(find simplebot_description)/meshes/roarm_m2/link5.stl"  scale="1.0 1.0 1.0"/>
-    </geometry>
-    <material name="silver"/>
-  </visual>
-  <collision>
-    <origin xyz="0 0 0" rpy="0 0 0" />
-    <geometry>
-      <mesh filename="file://$(find simplebot_description)/meshes/roarm_m2/link5.stl"  scale="1.0 1.0 1.0"/>
-    </geometry>
-  </collision>
-</link>
-<link name="gripper">
-  <inertial>
-    <origin xyz="0.0 0 0.0" rpy="0 0 0" />
-    <mass value="0.0028708" />
-    <inertia ixx="5.23216E-07" ixy="0" ixz="0" iyy="1.82071E-06" iyz="0" izz="1.60231E-06" />
-  </inertial>
-  <visual>
-    <origin xyz="0 0 0" rpy="0 0 0" />
-    <geometry>
-      <mesh filename="file://$(find simplebot_description)/meshes/roarm_m2/Gripper-B.stl"  scale="1.0 1.0 1.0"/>
-    </geometry>
-    <material name="silver"/>
-  </visual>
-  <collision>
-    <origin xyz="0 0 0" rpy="0 0 0" />
-    <geometry>
-      <mesh filename="file://$(find simplebot_description)/meshes/roarm_m2/Gripper-B.stl"  scale="1.0 1.0 1.0"/>
-    </geometry>
-  </collision>
-</link>
--->
+<!-- ===== ARM JOINTS ===== -->
 <joint name="roarm_base_link_to_link1" type="revolute">
   <origin xyz="0.0100000008759151 0 0.123059270461044" rpy="0 0 0" />
@@ -247,32 +132,24 @@
   <limit lower="-1" upper="2.95" effort="1000" velocity="1.0" />
 </joint>
-<joint name="link3_to_gripper_link" type="revolute">
- <origin xyz="-0.003266 -0.21599 -0.00560" rpy="3.1416 0 -1.5708" />
+<joint name="link3_to_link4" type="revolute">
+  <origin xyz="-0.003266 -0.21599 -0.00560" rpy="3.1416 0 -1.5708" />
   <parent link="link3" />
-  <child link="gripper_link" />
+  <child link="link4" />
   <axis xyz="0 0 1" />
-  <limit lower="-1.5" upper="1.5" effort="0" velocity="0" />
+  <limit lower="-1.5" upper="1.5" effort="10" velocity="1.0" />
 </joint>
-<joint name="gripper_link_to_gripper_b" type="revolute">
- <origin xyz="0.09187 0.0079 -0.00078" rpy="0 0 1.5708" />
-  <parent link="gripper_link" />
-  <child link="gripper_b" />
-  <axis xyz="0 1 0" />
-  <limit lower="-1.5" upper="1.5" effort="0" velocity="0" />
+<!-- Fixed joint placing tool0 at the end of link3 (the tool mounting point) -->
+<joint name="link4_to_link5" type="revolute">
+  <origin xyz="0.09187 0.0079 -0.00078" rpy="0 1.5708 0" />
+  <parent link="link4" />
+  <child link="link5" />
+  <axis xyz="0 0 1" />
+  <limit lower="-1.5" upper="1.5" effort="10" velocity="1.0" />
 </joint>
-<joint name="left_finger_joint" type="prismatic">
-    <parent link="gripper_b"/>
-    <child link="left_finger"/>
-    <origin xyz="0.00946 -0.08494 -0.05312" rpy="0 0 0"/>
-    <axis xyz="0 0 1"/>
-    <limit lower="-0.02" upper="0.02" effort="10.0" velocity="0.1"/>
+<joint name="link4_to_tool0" type="fixed">
+  <origin xyz="0.09187 0.0079 -0.00078" rpy="0 1.5708 0" />
+  <parent link="link4" />
+  <child link="tool0" />
 </joint>
-<joint name="right_finger_joint" type="prismatic">
-    <parent link="gripper_b"/>
-    <child link="right_finger"/>
-    <origin xyz="0.00946 -0.08494 0.05312" rpy="0 0 0"/>
-    <axis xyz="0 0 1"/>
-    <limit lower="-0.02" upper="0.02" effort="10.0" velocity="0.1"/>
-    <mimic joint="left_finger_joint" multiplier="-1.0" offset="0.0"/>
-</joint>
+<xacro:roarm_gripper parent="link5"/>
 </robot>

Commit message: controller works in gazebo

File: ros_ws/src/simplebot_description/urdf/control_m2/roarm_m2.ros2_control.xacro (robot description, xacro)
@@ -51,7 +51,11 @@
             <joint name="straight_bracket_left_joint">
             <command_interface name="position"/>
+            <state_interface name="position">
+                <param name="initial_value">0.0</param>
+            </state_interface>
             <state_interface name="position"/>
             <state_interface name="velocity"/>
             </joint>
+            <!-- Mimic joint for the right bracket -->
             <joint name="straight_bracket_right_joint">
             <param name="mimic">straight_bracket_left_joint</param>

File: ros_ws/src/simplebot_description/urdf/roarm_m2/gripper.xacro (robot description, xacro)
@@ -91,19 +91,19 @@
   <link name="right_gear_arm">
     <inertial>
-      <origin xyz="-0.0432 0.0 -0.0" rpy="0 0 0" />
-      <mass value="0.0028708" />
-      <inertia ixx="5.23216E-07" ixy="0" ixz="0" iyy="1.82071E-06" iyz="0" izz="1.60231E-06" />
-    </inertial>
-    <visual>
+      <origin xyz="-0.0 0.0 -0.0" rpy="0 0 0" />
+      <mass value="0.0028708" />
+      <inertia ixx="5.23216E-07" ixy="0" ixz="0" iyy="1.82071E-06" iyz="0" izz="1.60231E-06" />
+    </inertial>
+    <visual>
+      <origin xyz="-0.0 0 0" rpy="0 0 0" />
+      <geometry>
+        <mesh filename="file://$(find simplebot_description)/meshes/roarm_m2/right_swing_arm.stl"  scale="1.0 1.0 1.0"/>
+      </geometry>
+      <material name="silver"/>
+    </visual>
+    <collision>
       <origin xyz="-0.0432 0 0" rpy="0 0 0" />
       <geometry>
-        <mesh filename="file://$(find simplebot_description)/meshes/roarm_m2/gear_arm.stl"  scale="1.0 1.0 1.0"/>
-      </geometry>
-      <material name="silver"/>
-    </visual>
-    <collision>
-      <origin xyz="-0.0432 0 0" rpy="0 0 0" />
-      <geometry>
-        <mesh filename="file://$(find simplebot_description)/meshes/roarm_m2/gear_arm.stl"  scale="1.0 1.0 1.0"/>
+        <mesh filename="file://$(find simplebot_description)/meshes/roarm_m2/right_swing_arm.stl"  scale="1.0 1.0 1.0"/>
       </geometry>
     </collision>
@@ -173,5 +173,5 @@
       <origin xyz="-0.0315 -0.00496 0.0215" rpy="0 0 0"/>
       <axis xyz="0 1 0"/>
-      <limit lower="-1.545" upper="0" effort="10" velocity="1.0"/>
+      <limit lower="0" upper="1.545" effort="10" velocity="1.0"/>
       <mimic joint="straight_bracket_left_joint" multiplier="-1.0" offset="0.0"/>
   </joint>
@@ -191,5 +191,5 @@
       <origin xyz="-0.0105 -0.00496 0.0425" rpy="0 0 0"/>
       <axis xyz="0 1 0"/>
-      <limit lower="-1.545" upper="0" effort="10" velocity="1.0"/>
+      <limit lower="0" upper="1.545" effort="10" velocity="1.0"/>
       <mimic joint="straight_bracket_left_joint" multiplier="-1.0" offset="0.0"/>
   </joint>
@@ -201,5 +201,5 @@
       <origin xyz="0.0432 0.0045 0.0" rpy="0 0 0"/>
       <axis xyz="0 1 0"/>
-      <limit lower="-1.545" upper="0" effort="10" velocity="1.0"/>
+      <limit lower="0" upper="1.545" effort="10" velocity="1.0"/>
       <mimic joint="straight_bracket_left_joint" multiplier="-1.0" offset="0.0"/>
   </joint>
