Commit message: arm + gripepr works with moveit

File: ros_ws/src/simplebot_description/urdf/femto_bolt/femto_bolt.urdf.xacro (robot description, xacro)
@@ -144,5 +144,5 @@
           <update_rate>30</update_rate>
           <visualize>true</visualize>
-          <topic>${prefix}/depth</topic>
+          <topic>${prefix}/depth/image_raw</topic>
           <gz_frame_id>${prefix}_depth_optical_frame</gz_frame_id>
         </sensor>

File: ros_ws/src/simplebot_description/urdf/roarm_m2/gripper.xacro (robot description, xacro)
@@ -122,5 +122,5 @@
       <material name="silver"/>
     </visual>
-    <collision>
+    <collision name="left_finger_collision">
       <origin xyz="0 0 0" rpy="0 0 0" />
       <geometry>
@@ -128,4 +128,13 @@
       </geometry>
     </collision>
+    <sensor name="left_finger_contact" type="contact">
+      <contact>
+        <collision>left_finger_collision</collision>
+      </contact>
+      <always_on>1</always_on>
+      <update_rate>50</update_rate>
+      <visualize>true</visualize>
+      <topic>/gripper/left_contact</topic>
+    </sensor>
   </link>
   <link name="right_finger">
@@ -142,10 +151,19 @@
       <material name="silver"/>
     </visual>
-    <collision>
-      <origin xyz="0 0 0" rpy="0 0 0" />
-      <geometry>
-        <mesh filename="file://$(find simplebot_description)/meshes/roarm_m2/right_finger.stl"  scale="1.0 1.0 1.0"/>
-      </geometry>
-    </collision>
+    <collision name="right_finger_collision">
+      <origin xyz="0 0 0" rpy="0 0 0" />
+      <geometry>
+        <box size="0.01 0.01 0.05" />
+      </geometry>
+    </collision>
+    <sensor name="right_finger_contact" type="contact">
+      <contact>
+        <collision>right_finger_collision</collision>
+      </contact>
+      <always_on>1</always_on>
+      <update_rate>50</update_rate>
+      <visualize>true</visualize>
+      <topic>/gripper/right_contact</topic>
+    </sensor>
   </link>
   <!-- ===== GRIPPER JOINTS ===== -->
@@ -215,4 +233,10 @@
       <mimic joint="straight_bracket_left_joint" multiplier="1.0" offset="0.0"/>
   </joint>
+  <link name="hand_tcp"/>
+  <joint name="gripper_base_to_hand_tcp" type="fixed">
+    <origin xyz="0 -0.005 0.12" rpy="1.5708 0 0"/>
+    <parent link="gripper_base"/>
+    <child link="hand_tcp"/>
+  </joint>
 </xacro:macro>
 </robot>

File: ros_ws/src/simplebot_gripper_moveit_config/config/simplebot2.ros2_control.xacro (robot description, xacro)
@@ -29,8 +29,22 @@
                 <state_interface name="velocity"/>
             </joint>
-            <joint name="link3_to_gripper_link">
+            <joint name="link3_to_link4">
                 <command_interface name="position"/>
                 <state_interface name="position">
-                  <param name="initial_value">${initial_positions['link3_to_gripper_link']}</param>
+                  <param name="initial_value">${initial_positions['link3_to_link4']}</param>
+                </state_interface>
+                <state_interface name="velocity"/>
+            </joint>
+            <joint name="link4_to_link5">
+                <command_interface name="position"/>
+                <state_interface name="position">
+                  <param name="initial_value">${initial_positions['link4_to_link5']}</param>
+                </state_interface>
+                <state_interface name="velocity"/>
+            </joint>
+            <joint name="straight_bracket_left_joint">
+                <command_interface name="position"/>
+                <state_interface name="position">
+                  <param name="initial_value">${initial_positions['straight_bracket_left_joint']}</param>
                 </state_interface>
                 <state_interface name="velocity"/>

File: ros_ws/src/simplebot_gripper_moveit_config/config/simplebot2.urdf.xacro (robot description, xacro)
@@ -1,9 +1,9 @@
 <?xml version="1.0"?>
 <robot xmlns:xacro="http://www.ros.org/wiki/xacro" name="simplebot2">
-    <!-- <xacro:arg name="initial_positions_file" default="initial_positions.yaml" /> -->
+    <!--<xacro:arg name="initial_positions_file" default="initial_positions.yaml" /> -->
     <!-- Import simplebot2 urdf file -->
     <xacro:include filename="$(find simplebot_description)/urdf/robots/simplebot_description.urdf.xacro" />
     <!-- Import control_xacro -->
-    <!-- <xacro:include filename="simplebot2.ros2_control.xacro" /> -->
+    <!--<xacro:include filename="simplebot2.ros2_control.xacro" /> -->
     <!-- <xacro:simplebot2_ros2_control name="FakeSystem" initial_positions_file="$(arg initial_positions_file)"/> -->
 </robot>
