Commit message: Refactor SerialClient and RoArmHardware classes; add roarm_teleop package with joystick control

File: ros_ws/src/simplebot_description/urdf/control/simplebot_ros2_control.urdf.xacro (robot description, xacro)
@@ -4,12 +4,13 @@
         <ros2_control name="RobotSystem" type="system">
             <hardware>
-                <xacro:if value="${use_gazebo}">
+                <!-- <xacro:if value="${use_gazebo}"> -->
+                <xacro:if value="1">
                     <plugin>gz_ros2_control/GazeboSimSystem</plugin>
                 </xacro:if>
-                <xacro:unless value="${use_gazebo}">
+                <!-- <xacro:unless value="${use_gazebo}">
                     <plugin>simplebot_hardware/SimplebotChassisHardware</plugin>
                     <param name="serial_port">/dev/motor_controller</param>
                     <param name="baud_rate">115200</param>
-                </xacro:unless>
+                </xacro:unless>-->
             </hardware>
             <joint name="${prefix}front_left_wheel_joint">

File: ros_ws/src/simplebot_description/urdf/control_m2/roarm_m2.ros2_control.xacro (robot description, xacro)
@@ -52,10 +52,9 @@
             </joint>
             <joint name="straight_bracket_left_joint">
-            <command_interface name="position"/>
-            <state_interface name="position">
-                <param name="initial_value">0.0</param>
-            </state_interface>
-            <state_interface name="position"/>
-            <state_interface name="velocity"/>
+                <command_interface name="position"/>
+                <state_interface name="position">
+                    <param name="initial_value">0.0</param>
+                </state_interface>
+                <state_interface name="velocity"/>
             </joint>
             <!-- Mimic joint for the right bracket -->

File: ros_ws/src/simplebot_description/urdf/roarm_m2/gripper.xacro (robot description, xacro)
@@ -183,5 +183,5 @@
       <origin xyz="0.0315 -0.00496 0.0215" rpy="0 0 0"/>
       <axis xyz="0 1 0"/>
-      <limit lower="-1.545" upper="0" effort="10" velocity="1.0"/>
+      <limit lower="-1.6" upper="0" effort="10" velocity="1.0"/>
   </joint>
   <!-- Right bracket: mirrors left bracket via meshing gears -->
@@ -191,5 +191,5 @@
       <origin xyz="-0.0315 -0.00496 0.0215" rpy="0 0 0"/>
       <axis xyz="0 1 0"/>
-      <limit lower="0" upper="1.545" effort="10" velocity="1.0"/>
+      <limit lower="0" upper="1.6" effort="10" velocity="1.0"/>
       <mimic joint="straight_bracket_left_joint" multiplier="-1.0" offset="0.0"/>
   </joint>
@@ -200,5 +200,5 @@
       <origin xyz="0.0105 -0.00496 0.0425" rpy="0 0 0"/>
       <axis xyz="0 1 0"/>
-      <limit lower="-1.545" upper="0" effort="10" velocity="1.0"/>
+      <limit lower="-1.6" upper="0" effort="10" velocity="1.0"/>
       <mimic joint="straight_bracket_left_joint" multiplier="1.0" offset="0.0"/>
   </joint>
@@ -209,5 +209,5 @@
       <origin xyz="-0.0105 -0.00496 0.0425" rpy="0 0 0"/>
       <axis xyz="0 1 0"/>
-      <limit lower="0" upper="1.545" effort="10" velocity="1.0"/>
+      <limit lower="0" upper="1.6" effort="10" velocity="1.0"/>
       <mimic joint="straight_bracket_left_joint" multiplier="-1.0" offset="0.0"/>
   </joint>
@@ -219,5 +219,5 @@
       <origin xyz="0.0432 0.0045 0.0" rpy="0 0 0"/>
       <axis xyz="0 1 0"/>
-      <limit lower="0" upper="1.545" effort="10" velocity="1.0"/>
+      <limit lower="0" upper="1.6" effort="10" velocity="1.0"/>
       <mimic joint="straight_bracket_left_joint" multiplier="-1.0" offset="0.0"/>
   </joint>
@@ -230,5 +230,5 @@
       <origin xyz="-0.0432 0.0045 0.0" rpy="0 0 0"/>
       <axis xyz="0 1 0"/>
-      <limit lower="-1.545" upper="0" effort="10" velocity="1.0"/>
+      <limit lower="-1.6" upper="0" effort="10" velocity="1.0"/>
       <mimic joint="straight_bracket_left_joint" multiplier="1.0" offset="0.0"/>
   </joint>

File: ros_ws/src/simplebot_description/urdf/roarm_m2/roarm_m2.xacro (robot description, xacro)
@@ -90,4 +90,5 @@
 <link name="tool0" />
 <link name="link5" />
+<link name="base_link" />
 <link name="link4">
   <inertial>
@@ -111,4 +112,9 @@
 </link>
 <!-- ===== ARM JOINTS ===== -->
+<joint name="base_link_to_roarm_base_link" type="fixed">
+  <origin xyz="0.0 0 0.0" rpy="0 0 0" />
+  <parent link="base_link" />
+  <child link="roarm_base_link" />
+</joint>
 <joint name="roarm_base_link_to_link1" type="revolute">
   <origin xyz="0.0100000008759151 0 0.123059270461044" rpy="0 0 0" />
